Commit message: added new urdf

File: urdf/xArm.urdf (robot description, URDF)
Before this commit: robot roverarm, 15 links, 14 joints
Links:
- removed link arm_to_brover_link
- removed link base_footprint
- removed link base_scan
- removed link imu_link
- removed link wheel_left_link
- removed link wheel_right_link
- added link world
- link base_link: geometry 
Joints:
- removed joint arm_to_brover_joint
- removed joint base_joint
- removed joint imu_joint
- removed joint scan_joint
- removed joint wheel_left_joint
- removed joint wheel_right_joint
- added joint world_joint: type fixed, parent world, child base_link, origin xyz=0.0 0.0 0.05 rpy=0.0 0.0 0.0
- joint arm1: limit lower=-3.42 upper=0.7 effort=100 velocity=1.0 -> (none); origin xyz=0.0 0.0 0.06 rpy=0.0 0.0 0.0 -> xyz=0.0 0.0 0.05 rpy=0.0 0.0 0.0; parent arm_to_brover_link -> base_link; type revolute -> continuous
- joint arm2: limit lower=-1.51 upper=1.51 effort=100 velocity=1.0 -> (none); type revolute -> continuous
- joint arm3: limit lower=-2.12 upper=2.01 effort=100 velocity=1.0 -> (none); type revolute -> continuous
- joint arm4: limit lower=-1.92 upper=2.15 effort=100 velocity=1.0 -> (none); type revolute -> continuous
- joint arm5: limit lower=-0.46 upper=3.73 effort=100 velocity=1.0 -> (none); type revolute -> continuous

File: urdf/xArm_rover.urdf (robot description, URDF)
Before this commit: robot xArm, 10 links, 9 joints
Links:
- removed link world
- added link arm_to_brover_link; visual box size=0.1 0.1 0.005
- added link base_footprint
- added link base_scan; collision cylinder length=0.0315 radius=0.055; visual cylinder length=0.0315 radius=0.035
- added link imu_link; visual box size=0.18 0.18 0.002
- added link wheel_left_link; visual cylinder length=0.065 radius=0.06; visual cylinder length=0.065 radius=0.06
- added link wheel_right_link; visual cylinder length=0.065 radius=0.06; visual cylinder length=0.065 radius=0.06
- link base_link: geometry visual box size=0.405 0.28 0.115
Joints:
- removed joint world_joint
- added joint arm_to_brover_joint: type fixed, parent base_link, child arm_to_brover_link, origin xyz=0.15 -0.05 -0.015 rpy=0 1.57 0
- added joint base_joint: type fixed, parent base_footprint, child base_link, origin xyz=0.0 0.0 0.125 rpy=0 0 0
- added joint imu_joint: type fixed, parent base_link, child imu_link, origin xyz=0.15 0 0.025 rpy=0 0 0
- added joint scan_joint: type fixed, parent base_link, child base_scan, origin xyz=0.1 -0.065 0.08 rpy=0 0 3.1415
- added joint wheel_left_joint: type fixed, parent base_link, child wheel_left_link, origin xyz=0 0.215 -0.065 rpy=0 0 0, axis 0 0 1
- added joint wheel_right_joint: type fixed, parent base_link, child wheel_right_link, origin xyz=0 -0.215 -0.065 rpy=0 0 0, axis 0 0 1
- joint arm1: limit (none) -> lower=-3.42 upper=0.7 effort=100 velocity=1.0; origin xyz=0.0 0.0 0.05 rpy=0.0 0.0 0.0 -> xyz=0.0 0.0 0.06 rpy=0.0 0.0 0.0; parent base_link -> arm_to_brover_link; type continuous -> revolute
- joint arm2: limit (none) -> lower=-1.51 upper=1.51 effort=100 velocity=1.0; type continuous -> revolute
- joint arm3: limit (none) -> lower=-2.12 upper=2.01 effort=100 velocity=1.0; type continuous -> revolute
- joint arm4: limit (none) -> lower=-1.92 upper=2.15 effort=100 velocity=1.0; type continuous -> revolute
- joint arm5: limit (none) -> lower=-0.46 upper=3.73 effort=100 velocity=1.0; type continuous -> revolute
